File: GCController23-0899D/GCController23-0899D.kicad_pcb (KiCad board)
At the start: 4 copper layers, 135.1 x 98 mm, 80 parts, among them J1 Controller Connector, J2 C Stick Jumper, J3 C Stick Jumper, J4 L, J5 R, J7 R Analog, J8 L Analog, Q1 2SB0970, Q2 2SD1781K, Q3 2SC3757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

Commit message: added open source logo :smile:
Parts:
- added REF**: OSHW-Logo2_14.6x12mm_SilkScreen, Symbol:OSHW-Logo2_14.6x12mm_SilkScreen, B.Cu at (129.3, 63.5)
